File: PCB/Stimulator/Multi Chromatic Stimulator.kicad_pcb (KiCad board)
At the start: 2 copper layers, 125 x 75 mm, 43 parts, among them J2 5V - 30V

Commit message: PCB update
Parts:
- added ?: , , F.Cu at (79.3, 122.0)
- added ?: , , F.Cu at (19.8, -10.7)
- moved ? 1.60 mm to (135.3, 104.5)
Other:
- board text added: "Voltage Divider"
Changed lines of the file:
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@@
     (tracks 325)
     (zones 0)
-    (modules 43)
+    (modules 45)
     (nets 41)
   )
@@
     (add_net "Net-(Q1-Pad2)")
   )
+  (module "" (layer F.Cu)
+    (at 79.35 122.05)
+    (fp_text reference "" (at 19.8 -10.65) (layer F.SilkS)
+      (effects (font (size 1.27 1.27) (thickness 0.15)))
+    )
+    (fp_text value "" (at 19.8 -10.65) (layer F.SilkS)
+      (effects (font (size 1.27 1.27) (thickness 0.15)))
+    )
+    (fp_text user 5V (at 19.35 -18.85) (layer F.SilkS)
+      (effects (font (size 1 1) (thickness 0.15)))
+    )
+  )
+  (module "" (layer F.Cu)
+    (at 19.8 -10.65)
+    (fp_text reference "" (at 95.85 103.2) (layer F.SilkS)
+      (effects (font (size 1.27 1.27) (thickness 0.15)))
+    )
+    (fp_text value "" (at 95.85 103.2) (layer F.SilkS)
+      (effects (font (size 1.27 1.27) (thickness 0.15)))
+    )
+    (fp_text user 3.3V (at 79.35 118.95) (layer F.SilkS)
+      (effects (font (size 1 1) (thickness 0.15)))
+    )
+  )
   (module Connector_PinHeader_2.54mm:PinHeader_1x03_P2.54mm_Vertical (layer F.Cu)
     (at 95.85 103.2)
@@
   )
   (module "Maxime:new_logo 1000" (layer F.Cu)
-    (at 133.75 104.5)
+    (at 135.35 104.55)
     (fp_text reference "" (at 0 0) (layer F.SilkS) hide
       (effects (font (size 1.524 1.524) (thickness 0.3)))
@@
     )
   )
-  (gr_text "Signal \nInverter" (at 96.25 99.05) (layer F.SilkS)
+  (gr_text "Voltage\nDivider" (at 96.25 99.05) (layer F.SilkS)
     (effects (font (size 1.1 1.1) (thickness 0.25)))
   )
@@
   (segment (start 97.062081 105.75) (end 103.25 105.75) (width 0.25) (layer F.Cu) (net 6))
   (segment (start 95.85 102.604998) (end 95.85 103.2) (width 0.25) (layer F.Cu) (net 6))
+  (segment (start 78.85 105.7) (end 78.85 114.2) (width 0.25) (layer F.Cu) (net 6))
+  (segment (start 86.03 98.52) (end 78.85 105.7) (width 0.25) (layer F.Cu) (net 6))
+  (segment (start 86.03 98.52) (end 90.1 98.52) (width 0.25) (layer F.Cu) (net 6))
+  (segment (start 91.23137 98.52) (end 90.1 98.52) (width 0.25) (layer F.Cu) (net 6))
+  (segment (start 92.27 98.52) (end 91.23137 98.52) (width 0.25) (layer F.Cu) (net 6))
+  (segment (start 95.85 102.1) (end 92.27 98.52) (width 0.25) (layer F.Cu) (net 6))
+  (segment (start 95.85 103.2) (end 95.85 102.1) (width 0.25) (layer F.Cu) (net 6))
+  (segment (start 87.57 95.99) (end 87.57 94.83) (width 0.25) (layer F.Cu) (net 6))
+  (segment (start 90.1 98.52) (end 87.57 95.99) (width 0.25) (layer F.Cu) (net 6))
   (segment (start 91.850001 94.030001) (end 92.65 94.83) (width 0.25) (layer F.Cu) (net 8))
   (segment (start 90.964999 93.144999) (end 91.850001 94.030001) (width 0.25) (layer F.Cu) (net 8))
@@
   (segment (start 174.9 53.6) (end 179.5 49) (width 0.25) (layer F.Cu) (net 38))
   (segment (start 170.25 53.6) (end 174.9 53.6) (width 0.25) (layer F.Cu) (net 38))
-  (segment (start 78.85 105.7) (end 78.85 114.2) (width 0.25) (layer F.Cu) (net 6))
-  (segment (start 86.03 98.52) (end 78.85 105.7) (width 0.25) (layer F.Cu) (net 6))
-  (segment (start 86.03 98.52) (end 90.1 98.52) (width 0.25) (layer F.Cu) (net 6))
-  (segment (start 91.23137 98.52) (end 90.1 98.52) (width 0.25) (layer F.Cu) (net 6))
-  (segment (start 92.27 98.52) (end 91.23137 98.52) (width 0.25) (layer F.Cu) (net 6))
-  (segment (start 95.85 102.1) (end 92.27 98.52) (width 0.25) (layer F.Cu) (net 6))
-  (segment (start 95.85 103.2) (end 95.85 102.1) (width 0.25) (layer F.Cu) (net 6))
-  (segment (start 87.57 95.99) (end 87.57 94.83) (width 0.25) (layer F.Cu) (net 6))
-  (segment (start 90.1 98.52) (end 87.57 95.99) (width 0.25) (layer F.Cu) (net 6))
   (segment (start 94.17 65.1) (end 94.37 65.3) (width 0.25) (layer F.Cu) (net 39))
   (segment (start 90.65 65.1) (end 94.17 65.1) (width 0.25) (layer F.Cu) (net 39))

Commit message: update 24/10/2019
Other:
- board text added: "2019.09.18"
- board text added: "Multi-Chromatic Stimulator v2.2"
- board text removed: "2019.05.22"
- board text removed: "Multi-Chromatic Stimulator v2.1"
Changed lines of the file:
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@@
     (effects (font (size 1.5 1.5) (thickness 0.3)))
   )
-  (gr_text "Multi-Chromatic Stimulator v2.1" (at 134.5 57) (layer F.SilkS)
+  (gr_text "Multi-Chromatic Stimulator v2.2" (at 134.5 57) (layer F.SilkS)
     (effects (font (size 3.25 3.25) (thickness 0.5)))
   )
@@
     (effects (font (size 1.5 1.5) (thickness 0.3)) (justify left))
   )
-  (gr_text 2019.05.22 (at 168.5 60.7) (layer F.SilkS)
+  (gr_text 2019.09.18 (at 168.5 60.7) (layer F.SilkS)
     (effects (font (size 1.5 1.5) (thickness 0.3)))
   )
