File: PCB/Stimulator/LED Zappelin.kicad_pcb (KiCad board)
At the start: 2 copper layers, 125 x 75 mm, 45 parts, among them J2 5V - 30V

Commit message: Update PCB
Other:
- board text added: "2019.09.18"
- board text added: "LED Zappelin' v2.2"
- board text added: "by MJY Zimmermann Released under CERN OHL v1.2"
- board text removed: "2019.05.22"
- board text removed: "Multi-Chromatic Stimulator v2.1"
- board text removed: "by MJY Zimmermann & P Bartel Released under CERN OHL v1.2"
Changed lines of the file:
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@@
     (visible_elements 7FFFFFFF)
     (pcbplotparams
-      (layerselection 0x010fc_ffffffff)
+      (layerselection 0x3ffff_ffffffff)
       (usegerberextensions false)
       (usegerberattributes false)
@@
     (effects (font (size 1.5 1.5) (thickness 0.3)))
   )
-  (gr_text "Multi-Chromatic Stimulator v2.1" (at 134.5 57) (layer F.SilkS)
+  (gr_text "LED Zappelin' v2.2" (at 137.45 59.05) (layer F.SilkS)
     (effects (font (size 3.25 3.25) (thickness 0.5)))
   )
@@
     (effects (font (size 1.4 1.4) (thickness 0.25)) (justify left))
   )
-  (gr_text "by MJY Zimmermann & P Bartel\nReleased under CERN OHL v1.2" (at 129.35 65.2) (layer F.SilkS)
-    (effects (font (size 1.5 1.5) (thickness 0.3)) (justify left))
+  (gr_text "by MJY Zimmermann\nReleased under CERN OHL v1.2" (at 161.95 64.8) (layer F.SilkS)
+    (effects (font (size 1.5 1.5) (thickness 0.3)) (justify right))
   )
-  (gr_text 2019.05.22 (at 168.5 60.7) (layer F.SilkS)
+  (gr_text 2019.09.18 (at 168.5 60.7) (layer F.SilkS)
     (effects (font (size 1.5 1.5) (thickness 0.3)))
   )

Commit message: PCB update
Parts:
- ?: value 1k -> 150
Connections:
- ? pad 3V: Net-(A1-Pad16) -> (no net)
- ? pad USB: (no net) -> Net-(A1-Pad16)
Routing:
- net Net-(A1-Pad16): track 55.4 -> 64.9 mm
Changed lines of the file:
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@@
       (effects (font (size 1 1) (thickness 0.15)))
     )
-    (fp_text value 1k (at 6 0 180) (layer F.SilkS)
+    (fp_text value 150 (at 6 0 180) (layer F.SilkS)
       (effects (font (size 1 1) (thickness 0.15)))
     )
@@
     (pad SCK/5 thru_hole oval (at 21.83 -28.9 270) (size 1.6 1.6) (drill 0.8) (layers *.Cu *.Mask)
       (net 8 "Net-(A1-Pad25)"))
-    (pad USB thru_hole oval (at 1.5 -18.74 270) (size 1.6 1.6) (drill 0.8) (layers *.Cu *.Mask))
+    (pad USB thru_hole oval (at 1.5 -18.74 270) (size 1.6 1.6) (drill 0.8) (layers *.Cu *.Mask)
+      (net 13 "Net-(A1-Pad16)"))
     (pad MOSI/18 thru_hole oval (at 21.83 -31.44 270) (size 1.6 1.6) (drill 0.8) (layers *.Cu *.Mask)
       (net 9 "Net-(A1-Pad26)"))
@@
     (pad 21 thru_hole oval (at 21.83 -41.5 270) (size 1.6 1.6) (drill 0.8) (layers *.Cu *.Mask)
       (net 12 "Net-(A1-Pad30)"))
-    (pad 3V thru_hole oval (at 21.83 -6.04 270) (size 1.6 1.6) (drill 0.8) (layers *.Cu *.Mask)
-      (net 13 "Net-(A1-Pad16)"))
+    (pad 3V thru_hole oval (at 21.83 -6.04 270) (size 1.6 1.6) (drill 0.8) (layers *.Cu *.Mask))
     (pad RST thru_hole oval (at 21.83 -3.5 270) (size 1.6 1.6) (drill 0.8) (layers *.Cu *.Mask))
     (model ${KISYS3DMOD}/Module.3dshapes/Arduino_Nano_WithMountingHoles.wrl
@@
   (segment (start 105.25 84.5) (end 109.5 80.25) (width 0.25) (layer B.Cu) (net 12))
   (segment (start 105.25 94.83) (end 105.25 84.5) (width 0.25) (layer B.Cu) (net 12))
-  (segment (start 69.79 92.8) (end 69.23 92.24) (width 0.25) (layer F.Cu) (net 13))
-  (segment (start 69.79 94.83) (end 69.79 92.8) (width 0.25) (layer F.Cu) (net 13))
   (segment (start 63.25 86.26) (end 69.23 92.24) (width 0.25) (layer F.Cu) (net 13))
   (segment (start 63.25 76.4) (end 63.25 86.26) (width 0.25) (layer F.Cu) (net 13))
@@
   (segment (start 94.47 70.6) (end 94.47 71.73137) (width 0.25) (layer F.Cu) (net 13))
   (segment (start 94.47 71.73137) (end 93.90137 72.3) (width 0.25) (layer F.Cu) (net 13))
+  (segment (start 84.69 72.3) (end 93.90137 72.3) (width 0.25) (layer F.Cu) (net 13))
+  (segment (start 82.49 74.5) (end 84.69 72.3) (width 0.25) (layer F.Cu) (net 13))
   (segment (start 122.935 91.44) (end 124.095 91.44) (width 0.25) (layer B.Cu) (net 14))
   (segment (start 99.5 114.875) (end 122.935 91.44) (width 0.25) (layer B.Cu) (net 14))
